File: hardware/ephemerkey/mcu.kicad_sch (KiCad schematic)
At the start: 29 parts, among them J1 SWD TC2030-NL, J2 LOCK IF (I2C JST-PH), Q2 AO3400A, SW1 USER1, SW2 USER2, SW3 USER3/DFU, U1 STM32U083KCU6, Y1 32.768kHz

Commit message: hardware: gate OLED/EEPROM/I2C1 pull-ups behind PERI_EN load switch
Free the LIS3DH 2nd interrupt pin (tamper/free-fall now OR'd onto INT1 via
CTRL_REG3 I1_IA2) and repurpose it as PERI_EN. Add a high-side load switch on
the Sensors sheet (Q3 AO3401A pass FET, Q4 AO3400A gate driver, R30/R31 100k,
C31 1uF) powering a new +3V3_SW rail for DS1 OLED, U7 EEPROM, and the I2C1
pull-ups R9/R10 -- all gated off in Stop so they don't leak. LIS3DH stays on
always-on +3V3 as the wake source; FW drives PB6/PB7 low before Stop so the
powered accel never floats on the unpulled bus.

Surgical edits to both the .kicad_sch sheets and the schgen manifests (no
regen -- sheets are already partially wired). PARTS.md updated (also fills the
previously-missing Q2 AO3400A row). Also fix the lock J2 note: pin 2 = VCC <-
ephemerkey VSYS (was mislabeled "No-Connect", contradicting the wired net).

Co-Authored-By: Claude Opus 4.8 (1M context) <noreply@anthropic.com>
Changed lines of the file:
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@@
 		(company "EphemerKey Authors")
 	)
-	(text "MCU / RTC / Programming — pinout (U1 STM32U083KCU6, UFQFPN-32).  PLACED, not wired.\n pin  name            net / function           pin  name            net / function\n  1   VDD             +3V3  (C3 100nF)           17  VDDUSB          +3V3  (C5 100nF)\n  2   PC14/OSC32_IN   Y1 LSE 32.768kHz           18  PA8             GNSS_EN  -> GNSS\n  3   PC15/OSC32_OUT  Y1 LSE 32.768kHz           19  PA9             USART1_TX -> GNSS RXD\n  4   PF2/NRST        NRST (C9 100nF, J1)        20  PA10            USART1_RX <- GNSS TXD\n  5   VDDA/VREF+      +3V3 (C7 1uF, C8 100nF)    21  PA11            USB_DM   (<- U3 ESD)\n  6   PA0             GNSS_PPS (TIM2_CH1 in)     22  PA12            USB_DP   (<- U3 ESD)\n  7   PA1             GNSS_EXTINT (out)          23  PA13            SWDIO (J1)\n  8   PA2             ACC_INT1 (EXTI wake)       24  PA14            SWCLK (J1)\n  9   PA3             ACC_INT2 (EXTI tamper)     25  PA15            BTN2 SW2 (pull-up)\n 10   PA4             GNSS_RESET_N (OD out)      26  PB3             spare\n 11   PA5             BTN1 SW1 (pull-up->GND)    27  PB4             BUZZER_PWM (TIM3_CH1) -> R13 -> Q2\n 12   PA6             LED_GRN  D1 + R2 1k        28  PB5             spare\n 13   PA7             LED_RED  D2 + R3 1k        29  PB6             I2C1_SCL -> U5\n 14   PB0             LOCK_SDA <> J2.3 (I2C R11)  30  PB7             I2C1_SDA -> U5\n 15   PB1             LOCK_SCL -> J2.4 (I2C R12)  31  PF3/BOOT0       BTN3 SW3 + DFU\n 16   VSS             GND                        32  VSS  / EP       GND\nRTC:  Y1 32.768kHz across PC14/PC15; C1,C2 12pF load caps (match to Y1 CL; trim via RTC SMOOTHCALIB).\nBUZZER:  LS1 MLT-8530 (3.6V magnetic transducer, ~2.7kHz, 95mA): pin1 = +3V3, pin2 = BUZZ_DRV (Q2 drain).\n      Q2 AO3400A low-side: G <- R13 100R <- BUZZER_PWM (PB4/TIM3_CH1); S -> GND; D -> BUZZ_DRV.  R14 100k gate->GND\n      (off-safe). D5 1N4148W flyback across LS1: A = BUZZ_DRV, K = +3V3.  FW drives PB4 PWM ~2.7kHz for tones.\nPWR:  +3V3 from PSU sheet, C6 10uF bulk.   J1 = SWD TC2030-NL: SWDIO, SWCLK, NRST, +3V3, GND.\nBTN:  3 user buttons. SW1->PA5, SW2->PA15 active-low (MCU pull-ups, to GND).\n      SW3->PF3/BOOT0 active-HIGH to +3V3 (R1 10k pulldown = default boot-from-flash).\n      Hold SW3 at reset (NRST via J1 / power cycle) -> ROM bootloader -> USB DFU over USB-C\n      (STM32U0 supports USB DFU, AN2606; crystal-less USB via HSI48+CRS).\nJ2 LOCK IF (RA JST-PH 4-pin, S4B-PH-K; AUTHENTICATED I2C; ephemerkey = MASTER, lock = TARGET; = hardware/lock):\n      1 = GND   2 = VSYS (battery/system rail -> POWERS the lock; the lock has NO own cell)   3 = LOCK_SDA   4 = LOCK_SCL.\n      The lock draws its logic + boost/actuator current from VSYS over this cable.  CAUTION: a 12V solenoid pull-in is\n      ~3-4A from VSYS -> exceeds JST-PH (~2A/contact) and ephemerkey's load-share path; keep actuation to the 6V servo /\n      low duty w/ the lock's reservoir caps, or run a heavier dedicated power feed to the lock.\n      Wake-on-I2C (no discrete line): lock wakes on SCL START; master sends a dummy/wake xfer then retries.\n      I2C pull-ups R11/R12 4.7k -> +3V3 (KEEP at 3V3: STM32 PB0/PB1 are not >3.6V tolerant -- do NOT pull to VSYS; the\n      lock's I2C VIH ~0.7*VSYS is met by a 3V3 bus across the discharge curve).  AUTH = HMAC-SHA1 (reuse smalltotp).\nDS1 OLED (1x4, 0.1in header, 128x32 I2C, 3V3):  1 = GND  2 = +3V3  3 = SCL (PB6)  4 = SDA (PB7).\n      Shares I2C1 with U5 (OLED 0x3C, LIS3DH 0x18); pull-ups R9/R10 on Sensors sheet serve both."
+	(text "MCU / RTC / Programming — pinout (U1 STM32U083KCU6, UFQFPN-32).  PLACED, not wired.\n pin  name            net / function           pin  name            net / function\n  1   VDD             +3V3  (C3 100nF)           17  VDDUSB          +3V3  (C5 100nF)\n  2   PC14/OSC32_IN   Y1 LSE 32.768kHz           18  PA8             GNSS_EN  -> GNSS\n  3   PC15/OSC32_OUT  Y1 LSE 32.768kHz           19  PA9             USART1_TX -> GNSS RXD\n  4   PF2/NRST        NRST (C9 100nF, J1)        20  PA10            USART1_RX <- GNSS TXD\n  5   VDDA/VREF+      +3V3 (C7 1uF, C8 100nF)    21  PA11            USB_DM   (<- U3 ESD)\n  6   PA0             GNSS_PPS (TIM2_CH1 in)     22  PA12            USB_DP   (<- U3 ESD)\n  7   PA1             GNSS_EXTINT (out)          23  PA13            SWDIO (J1)\n  8   PA2             ACC_INT1 (EXTI wake)       24  PA14            SWCLK (J1)\n  9   PA3             PERI_EN (periph pwr gate)  25  PA15            BTN2 SW2 (pull-up)\n 10   PA4             GNSS_RESET_N (OD out)      26  PB3             spare\n 11   PA5             BTN1 SW1 (pull-up->GND)    27  PB4             BUZZER_PWM (TIM3_CH1) -> R13 -> Q2\n 12   PA6             LED_GRN  D1 + R2 1k        28  PB5             spare\n 13   PA7             LED_RED  D2 + R3 1k        29  PB6             I2C1_SCL -> U5\n 14   PB0             LOCK_SDA <> J2.3 (I2C R11)  30  PB7             I2C1_SDA -> U5\n 15   PB1             LOCK_SCL -> J2.4 (I2C R12)  31  PF3/BOOT0       BTN3 SW3 + DFU\n 16   VSS             GND                        32  VSS  / EP       GND\nRTC:  Y1 32.768kHz across PC14/PC15; C1,C2 12pF load caps (match to Y1 CL; trim via RTC SMOOTHCALIB).\nBUZZER:  LS1 MLT-8530 (3.6V magnetic transducer, ~2.7kHz, 95mA): pin1 = +3V3, pin2 = BUZZ_DRV (Q2 drain).\n      Q2 AO3400A low-side: G <- R13 100R <- BUZZER_PWM (PB4/TIM3_CH1); S -> GND; D -> BUZZ_DRV.  R14 100k gate->GND\n      (off-safe). D5 1N4148W flyback across LS1: A = BUZZ_DRV, K = +3V3.  FW drives PB4 PWM ~2.7kHz for tones.\nPWR:  +3V3 from PSU sheet, C6 10uF bulk.   J1 = SWD TC2030-NL: SWDIO, SWCLK, NRST, +3V3, GND.\nBTN:  3 user buttons. SW1->PA5, SW2->PA15 active-low (MCU pull-ups, to GND).\n      SW3->PF3/BOOT0 active-HIGH to +3V3 (R1 10k pulldown = default boot-from-flash).\n      Hold SW3 at reset (NRST via J1 / power cycle) -> ROM bootloader -> USB DFU over USB-C\n      (STM32U0 supports USB DFU, AN2606; crystal-less USB via HSI48+CRS).\nJ2 LOCK IF (RA JST-PH 4-pin, S4B-PH-K; AUTHENTICATED I2C; ephemerkey = MASTER, lock = TARGET; = hardware/lock):\n      1 = GND   2 = VSYS (battery/system rail -> POWERS the lock; the lock has NO own cell)   3 = LOCK_SDA   4 = LOCK_SCL.\n      The lock draws its logic + boost/actuator current from VSYS over this cable.  CAUTION: a 12V solenoid pull-in is\n      ~3-4A from VSYS -> exceeds JST-PH (~2A/contact) and ephemerkey's load-share path; keep actuation to the 6V servo /\n      low duty w/ the lock's reservoir caps, or run a heavier dedicated power feed to the lock.\n      Wake-on-I2C (no discrete line): lock wakes on SCL START; master sends a dummy/wake xfer then retries.\n      I2C pull-ups R11/R12 4.7k -> +3V3 (KEEP at 3V3: STM32 PB0/PB1 are not >3.6V tolerant -- do NOT pull to VSYS; the\n      lock's I2C VIH ~0.7*VSYS is met by a 3V3 bus across the discharge curve).  AUTH = HMAC-SHA1 (reuse smalltotp).\nDS1 OLED (1x4, 0.1in header, 128x32 I2C, 3V3):  1 = GND  2 = +3V3_SW (GATED, Sensors Q3)  3 = SCL (PB6)  4 = SDA (PB7).\n      Shares I2C1 with U5 (OLED 0x3C, LIS3DH 0x18); pull-ups R9/R10 on Sensors sheet serve both."
 		(exclude_from_sim no)
 		(at 12 198.88 0)
