File: hardware/ephemerkey/sensors.kicad_sch (KiCad schematic)
At the start: 6 parts, among them U5 LIS3DHTR

Commit message: hardware: gate OLED/EEPROM/I2C1 pull-ups behind PERI_EN load switch
Free the LIS3DH 2nd interrupt pin (tamper/free-fall now OR'd onto INT1 via
CTRL_REG3 I1_IA2) and repurpose it as PERI_EN. Add a high-side load switch on
the Sensors sheet (Q3 AO3401A pass FET, Q4 AO3400A gate driver, R30/R31 100k,
C31 1uF) powering a new +3V3_SW rail for DS1 OLED, U7 EEPROM, and the I2C1
pull-ups R9/R10 -- all gated off in Stop so they don't leak. LIS3DH stays on
always-on +3V3 as the wake source; FW drives PB6/PB7 low before Stop so the
powered accel never floats on the unpulled bus.

Surgical edits to both the .kicad_sch sheets and the schgen manifests (no
regen -- sheets are already partially wired). PARTS.md updated (also fills the
previously-missing Q2 AO3400A row). Also fix the lock J2 note: pin 2 = VCC <-
ephemerkey VSYS (was mislabeled "No-Connect", contradicting the wired net).

Co-Authored-By: Claude Opus 4.8 (1M context) <noreply@anthropic.com>
Parts:
- added C31: 1uF, Capacitor_SMD:C_0402_1005Metric, symbol Device:C
- added Q3: AO3401A, Package_TO_SOT_SMD:SOT-23, symbol Transistor_FET:Q_PMOS_GSD
- added Q4: AO3400A, Package_TO_SOT_SMD:SOT-23, symbol Transistor_FET:Q_NMOS_GSD
- added R30, R31: 100k, Resistor_SMD:R_0402_1005Metric, symbol Device:R
Connections:
- net ACCEL_TAMPER renamed PERI_EN
Other:
- note added: "Sensors — pinout (U5 LIS3DHTR, LGA-16). PLACED, not wired. U5 LIS3DH: 1 VDD_IO +3V3 (C24 100nF) 9 INT2 NC (2nd alarm removed) 2 NC 10 RES -> GND 3 NC 11 INT1 -> PA2 (wake + tamper, OR via CTRL_REG3 I1_IA2) 4 SCL -> PB6 (I2C1) 12 GND GND 5 GND GND 13 ADC3 NC 6 SDA -> PB7 (I2C1) 14 VDD +3V3 (C23 100nF) 7 SDO/SA0 addr 0x18(GND)/0x19 15 ADC2 NC 8 CS +3V3 (force I2C) 16 ADC1 NC I2C1: R9/R10 4.7k pull-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"
- note removed: "Sensors — pinout (U5 LIS3DHTR, LGA-16). PLACED, not wired. U5 LIS3DH: 1 VDD_IO +3V3 (C24 100nF) 9 INT2 -> PA3 (tamper / free-fall) 2 NC 10 RES -> GND 3 NC 11 INT1 -> PA2 (wake-on-motion) 4 SCL -> PB6 (I2C1) 12 GND GND 5 GND GND 13 ADC3 NC 6 SDA -> PB7 (I2C1) 14 VDD +3V3 (C23 100nF) 7 SDO/SA0 addr 0x18(GND)/0x19 15 ADC2 NC 8 CS +3V3 (force I2C) 16 ADC1 NC I2C1: R9/R10 4.7k pull-ups to +3V3. Tamper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"
